Commit message: Week6_Done

File: install/arm_description/share/arm_description/urdf/simple_arm.urdf (robot description, URDF)
Before this commit: robot simple_arm, 3 links, 2 joints
Links:
- link link1: geometry collision cylinder length=0.5 radius=0.05; visual box size=0.2 0.06 0.5
- link link2: geometry collision cylinder length=0.4 radius=0.04; visual box size=0.2 0.06 0.5
